File: 25Zak001 ESP32 Mark0.kicad_sch (KiCad schematic)
At the start: 3 parts, among them J1 USB_C_Receptacle_PowerOnly_6P, U1 ESP32-C3-DevKitM-1, U2 ESP32_NODEMCU

Commit message: Pridano USB C
Parts:
- added H1, H2, H3, H4: MountingHole, MountingHole:MountingHole_3.2mm_M3_ISO14580_Pad_TopBottom, symbol Mechanical:MountingHole
- J1: footprint (none) -> Connector_USB:USB_C_Receptacle_GCT_USB4135-GF-A_6P_TopMnt_Horizontal

Commit message: Nova verze
Parts:
- removed U1: ESP32-C3-DevKitM-1, RF_Module:ESP32-C3-DevKitM-1, symbol RF_Module:ESP32-C3-DevKitM-1
- added J2: BME280, Connector_PinSocket_2.54mm:PinSocket_1x04_P2.54mm_Vertical, symbol Connector:Conn_01x04_Socket
- added J3: eInk display, Connector_PinSocket_2.54mm:PinSocket_1x09_P2.54mm_Horizontal, symbol Connector:Conn_01x08_Socket
- A1: renamed from U2; footprint ESP32_NODEMCU:MODULE_ESP32_NODEMCU -> ndoemcu:MODULE_ESP32_NODEMCU
Connections:
- net GND: now also A1.J4_1 (GND_1), A1.J4_7 (GND_7), A1.J5_6 (GND_6), J1.S1 (SHIELD), J2.2 (Pin_2), J3.7 (Pin_7)
- net CLK: now reaches A1.J4_19 (CLK)
- net CLK: now also J3.5 (Pin_5)
- new net BUSY: J3.1 (Pin_1)
- new net CS: J3.4 (Pin_4)
- new net DC: J3.3 (Pin_3)
- new net DIN: J3.6 (Pin_6)
- new net RST: J3.2 (Pin_2)
- new net SCL: J2.3 (Pin_3)
- new net SDA: J2.4 (Pin_4)
- new net VCC: J2.1 (Pin_1), J3.8 (Pin_8)

Commit message: Dokonceni, plno chyb, nutno opravit
Parts:
- removed A1: ESP32_NODEMCU, ndoemcu:MODULE_ESP32_NODEMCU, symbol moje_knihovna:ESP32_NODEMCU
- added J4: Conn_01x08_Pin, Connector_PinHeader_2.54mm:PinHeader_1x08_P2.54mm_Vertical, symbol Connector:Conn_01x08_Pin
- added J5: Conn_01x06_Pin, Connector_PinHeader_2.54mm:PinHeader_1x06_P2.54mm_Vertical, symbol Connector:Conn_01x06_Pin
- added NodeMCU-C6-DevkitM1: ~, ndoemcu:ESP32-C6-DevKitM-1, symbol moje_knihovna:NodeMCU_C6
Connections:
- net VCC is gone; now on net +5V: J2.1 (Pin_1), J3.8 (Pin_8)
- net BUSY: now also NodeMCU-C6-DevkitM1.17 (GPIO16)
- net CLK: now also NodeMCU-C6-DevkitM1.22 (GPIO20)
- net CS: now also NodeMCU-C6-DevkitM1.23 (GPIO19)
- net DC: now also NodeMCU-C6-DevkitM1.24 (GPIO18)
- net DIN: now also NodeMCU-C6-DevkitM1.21 (GPIO21)
- net GND: now also NodeMCU-C6-DevkitM1.13 (GND), NodeMCU-C6-DevkitM1.15 (GND), NodeMCU-C6-DevkitM1.16 (GND), NodeMCU-C6-DevkitM1.27 (GND), NodeMCU-C6-DevkitM1.30 (GND)
- net RST: now also NodeMCU-C6-DevkitM1.18 (GPIO17)
- net SCL: now also NodeMCU-C6-DevkitM1.9 (GPIO8)
- net SDA: now also NodeMCU-C6-DevkitM1.26 (GPIO9)
- net +5V: now reaches J1.A9 (VBUS), J1.B9 (VBUS)
- net +5V: now also NodeMCU-C6-DevkitM1.14 (+5V)
- new net +3.3V: NodeMCU-C6-DevkitM1.1 (3V3)
- new net GPIO0: J4.1 (Pin_1), NodeMCU-C6-DevkitM1.7 (GPIO0)
- new net GPIO1: J4.2 (Pin_2), NodeMCU-C6-DevkitM1.8 (GPIO1)
- new net GPIO12: J5.1 (Pin_1), NodeMCU-C6-DevkitM1.29 (GPIO12)
- new net GPIO13: J5.2 (Pin_2), NodeMCU-C6-DevkitM1.28 (GPIO13)
- new net GPIO14: J5.3 (Pin_3), NodeMCU-C6-DevkitM1.12 (GPIO14)
- new net GPIO15: J5.4 (Pin_4), NodeMCU-C6-DevkitM1.25 (GPIO15)
- new net GPIO2: J4.3 (Pin_3), NodeMCU-C6-DevkitM1.3 (GPIO2)
- new net GPIO22: J5.5 (Pin_5), NodeMCU-C6-DevkitM1.20 (GPIO22)
- new net GPIO23: J5.6 (Pin_6), NodeMCU-C6-DevkitM1.19 (GPIO23)
- new net GPIO3: J4.4 (Pin_4), NodeMCU-C6-DevkitM1.4 (GPIO3)
- new net GPIO4: J4.5 (Pin_5), NodeMCU-C6-DevkitM1.5 (GPIO4)
- new net GPIO5: J4.6 (Pin_6), NodeMCU-C6-DevkitM1.6 (GPIO5)
- new net GPIO6: J4.7 (Pin_7), NodeMCU-C6-DevkitM1.10 (GPIO6)
- new net GPIO7: J4.8 (Pin_8), NodeMCU-C6-DevkitM1.11 (GPIO7)
- no-connect marks 0 -> 2
Other:
- note added: "BME280 Module"
- note added: "NodeMCU ESP32 C6 Devkit M1"
- note added: "USB C - Power only"
- note added: "Unused GPIOs"
- note added: "eInk Display [SPI bus]"
- moved on the sheet: J2, J3
