File: 25Zak001 ESP32 Mark0.kicad_sch (KiCad schematic)
At the start: 11 parts, among them J1 USB_C_Receptacle_PowerOnly_6P, J2 eInk display SPI, J3 Free GPIOs from Left Side, J4 Free GPIOs from Right Side, J6 ESP32 Left Side, J7 ESP32 Right Side, U1 DHT11_muj

Commit message: Rev1 created for PCB
Because Rev0 is virutally unusable in current state.
Parts:
- J4: footprint (none) -> Connector_PinSocket_2.54mm:PinSocket_1x07_P2.54mm_Vertical
Other:
- company: (none) -> Zdenek Rusek
- title: (none) -> ESP32 Weather Station
Changed lines of the file:
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@@
 	(generator_version "9.0")
 	(paper "A4")
+	(title_block
+		(title "ESP32 Weather Station")
+		(rev "1")
+		(company "Zdenek Rusek")
+	)
 	(rectangle
 		(start 20.32 22.86)
@@
 			)
 		)
-		(property "Footprint" ""
+		(property "Footprint" "Connector_PinSocket_2.54mm:PinSocket_1x07_P2.54mm_Vertical"
 			(at 81.28 39.37 0)
 			(effects
