File: _autosave-25Zak001 ESP32 Mark0.kicad_sch (KiCad schematic)
At the start: 11 parts, among them J1 USB_C_Receptacle_PowerOnly_6P, J2 eInk display SPI, J3 Free GPIOs from Left Side, J4 Free GPIOs from Right Side, J6 ESP32 Left Side, J7 ESP32 Right Side, U1 DHT11_muj

Commit message: Fairly Big Update
- completly reworked ESP32 devkit
- different sensor
- all unused GPIOs are now available via sockets
Parts:
- J4: footprint (none) -> Connector_PinSocket_2.54mm:PinSocket_1x07_P2.54mm_Vertical
Changed lines of the file:
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@@
 			)
 		)
-		(property "Footprint" ""
+		(property "Footprint" "Connector_PinSocket_2.54mm:PinSocket_1x07_P2.54mm_Vertical"
 			(at 81.28 39.37 0)
 			(effects
